Commit message: Fix Allegro-left thumb mirror; add s01-u02 / s02 refs; update run list
- allegro_hand_left_6dof.urdf: mirror joint_13 origin y (0.005 -> -0.005),
  an incomplete-mirror bug; Allegro-left thumb now matches RH (~6-10 mm overall).
- Rebuild all Allegro/Inspire graph refs; add ketchup_use_02 (s01) and
  notebook_use_02 (s02) bimanual refs.
- runs_graph.tsv: switch to the 7 explicit paper clips
  (ketchup-30-130-s01-u01, box-30-230-s01-u01, mixer-30-200-s01-u01,
   ketchup-40-340-s01-u02, mixer-40-340-s01-u01, notebook-40-340-s02-u02,
   waffleiron-40-340-s01-u01).

Co-Authored-By: Claude Opus 4.8 <noreply@anthropic.com>

File: dexmachina/assets/allegro_hand/allegro_hand_left_6dof.urdf (robot description, URDF)
Before this commit: robot allegro_left, 29 links, 28 joints
Joints:
- joint joint_13.0: origin xyz=-0.027 0.005 0.0399 -> xyz=-0.027 -0.005 0.0399

Commit message: feat(oakink): port OakInk-v2 (two rigid objects/hand) for task+imitation RL
Generalize the ARCTIC-specialized env along the object axis (no-op when n_objects==1):
- rewards.py: per-object load_demo (demo_data['objects']) + precomputed_task hook.
- base_env.py: per-object demo wiring, per-object task reward (mean), dones over all
  objects, set_retarget_states sets both objects from demo (kinematic replay).
- object.py: get_oakink_object_cfg (rigid, frozen dummy joint, contact_sides).
- demo_data.py: nested per-object demo slicing in load_genesis_retarget_data.
- constructors.py: --oakink/--oakink_pt branch (_get_oakink_env_cfg), contacts off.
- rl/replay_oakink.py: kinematic set-state replay (headless check or --vis).
- retargeting/stage_oakink_objects.py: stage 106 OakInk objects as rigid URDFs.
- assets/oakink/: staged objects; assets/retargeted/allegro_hand/oakink/: sample kinref.

Contacts deferred (task+imitation milestone). Bundles related WIP it depends on:
robot.py RSI hand-reset for hybrid/absolute, allegro forearm limits +-12 rad.

Co-Authored-By: Claude Opus 4.8 (1M context) <noreply@anthropic.com>

File: dexmachina/assets/allegro_hand/allegro_hand_left_6dof.urdf (robot description, URDF)
Before this commit: robot allegro_left, 29 links, 28 joints
Joints:
- joint L_forearm_pitch_link_joint: limit lower=-6.2 upper=6.2 effort=100 velocity=5 -> lower=-12.0 upper=12.0 effort=100 velocity=5
- joint L_forearm_roll_link_joint: limit lower=-6.2 upper=6.2 effort=100 velocity=5 -> lower=-12.0 upper=12.0 effort=100 velocity=5
- joint L_forearm_yaw_link_joint: limit lower=-6.2 upper=6.2 effort=100 velocity=5 -> lower=-12.0 upper=12.0 effort=100 velocity=5

File: dexmachina/assets/allegro_hand/allegro_hand_right_6dof.urdf (robot description, URDF)
Before this commit: robot allegro_right, 29 links, 28 joints
Joints:
- joint R_forearm_pitch_link_joint: limit lower=-6.2 upper=6.2 effort=100 velocity=5 -> lower=-12.0 upper=12.0 effort=100 velocity=5
- joint R_forearm_roll_link_joint: limit lower=-6.2 upper=6.2 effort=100 velocity=5 -> lower=-12.0 upper=12.0 effort=100 velocity=5
- joint R_forearm_yaw_link_joint: limit lower=-6.2 upper=6.2 effort=100 velocity=5 -> lower=-12.0 upper=12.0 effort=100 velocity=5
