Commit message: perf(oakink): rigid objects as true free bodies (no dummy joint) -> ~4x faster sim
The frozen massless dummy revolute joint (mass 1e-6, + Genesis zeros its armature/damping)
made the articulated-body solver ill-conditioned -> OakInk sim ran ~4x slower than ARCTIC
(isolated to fps_step, contacts off). Regenerate the 106 OakInk URDFs as single-link free
rigid bodies (no joint); ArticulatedObject now treats 0 movable joints as rigid: keep
num_joints=1 VIRTUAL (buffers/obs/reward/state_diff shapes unchanged) but skip entity dof-I/O
(get/set_dofs) when dof_idxs is empty. ARCTIC (1 real joint) is byte-identical.

Co-Authored-By: Claude Opus 4.8 (1M context) <noreply@anthropic.com>

File: dexmachina/assets/oakink/C10001/object.urdf (robot description, URDF)
Before this commit: robot C10001, 2 links, 1 joints
Links:
- removed link tip_dummy
Joints:
- removed joint rotation

File: dexmachina/assets/oakink/C11001/object.urdf (robot description, URDF)
Before this commit: robot C11001, 2 links, 1 joints
Links:
- removed link tip_dummy
Joints:
- removed joint rotation

File: dexmachina/assets/oakink/C12001/object.urdf (robot description, URDF)
Before this commit: robot C12001, 2 links, 1 joints
Links:
- removed link tip_dummy
Joints:
- removed joint rotation

File: dexmachina/assets/oakink/C14001/object.urdf (robot description, URDF)
Before this commit: robot C14001, 2 links, 1 joints
Links:
- removed link tip_dummy
Joints:
- removed joint rotation

File: dexmachina/assets/oakink/C43001/object.urdf (robot description, URDF)
Before this commit: robot C43001, 2 links, 1 joints
Links:
- removed link tip_dummy
Joints:
- removed joint rotation

File: dexmachina/assets/oakink/C51001/object.urdf (robot description, URDF)
Before this commit: robot C51001, 2 links, 1 joints
Links:
- removed link tip_dummy
Joints:
- removed joint rotation

File: dexmachina/assets/oakink/O02_0003_00004/object.urdf (robot description, URDF)
Before this commit: robot O02_0003_00004, 2 links, 1 joints
Links:
- removed link tip_dummy
Joints:
- removed joint rotation

File: dexmachina/assets/oakink/O02_0003_00005/object.urdf (robot description, URDF)
Before this commit: robot O02_0003_00005, 2 links, 1 joints
Links:
- removed link tip_dummy
Joints:
- removed joint rotation

File: dexmachina/assets/oakink/O02_0010_00003/object.urdf (robot description, URDF)
Before this commit: robot O02_0010_00003, 2 links, 1 joints
Links:
- removed link tip_dummy
Joints:
- removed joint rotation

File: dexmachina/assets/oakink/O02_0011_00001/object.urdf (robot description, URDF)
Before this commit: robot O02_0011_00001, 2 links, 1 joints
Links:
- removed link tip_dummy
Joints:
- removed joint rotation

File: dexmachina/assets/oakink/O02_0011_00002/object.urdf (robot description, URDF)
Before this commit: robot O02_0011_00002, 2 links, 1 joints
Links:
- removed link tip_dummy
Joints:
- removed joint rotation

File: dexmachina/assets/oakink/O02_0011_00003/object.urdf (robot description, URDF)
Before this commit: robot O02_0011_00003, 2 links, 1 joints
Links:
- removed link tip_dummy
Joints:
- removed joint rotation

File: dexmachina/assets/oakink/O02_0013_00004/object.urdf (robot description, URDF)
Before this commit: robot O02_0013_00004, 2 links, 1 joints
Links:
- removed link tip_dummy
Joints:
- removed joint rotation

File: dexmachina/assets/oakink/O02_0013_00005/object.urdf (robot description, URDF)
Before this commit: robot O02_0013_00005, 2 links, 1 joints
Links:
- removed link tip_dummy
Joints:
- removed joint rotation

File: dexmachina/assets/oakink/O02_0015_00001/object.urdf (robot description, URDF)
Before this commit: robot O02_0015_00001, 2 links, 1 joints
Links:
- removed link tip_dummy
Joints:
- removed joint rotation

File: dexmachina/assets/oakink/O02_0015_00002/object.urdf (robot description, URDF)
Before this commit: robot O02_0015_00002, 2 links, 1 joints
Links:
- removed link tip_dummy
Joints:
- removed joint rotation

File: dexmachina/assets/oakink/O02_0015_00004/object.urdf (robot description, URDF)
Before this commit: robot O02_0015_00004, 2 links, 1 joints
Links:
- removed link tip_dummy
Joints:
- removed joint rotation

File: dexmachina/assets/oakink/O02_0015_00005/object.urdf (robot description, URDF)
Before this commit: robot O02_0015_00005, 2 links, 1 joints
Links:
- removed link tip_dummy
Joints:
- removed joint rotation

File: dexmachina/assets/oakink/O02_0015_00007/object.urdf (robot description, URDF)
Before this commit: robot O02_0015_00007, 2 links, 1 joints
Links:
- removed link tip_dummy
Joints:
- removed joint rotation

File: dexmachina/assets/oakink/O02_0015_00008/object.urdf (robot description, URDF)
Before this commit: robot O02_0015_00008, 2 links, 1 joints
Links:
- removed link tip_dummy
Joints:
- removed joint rotation
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